File: robo-roach-v1.0.kicad_sch (KiCad schematic)
At the start: 42 parts, among them J1 USB_C_Receptacle_PowerOnly_6P, J2 Prog, M1 Motor_DC, M2 Motor_DC, Q1 T2N7002AK, SW1 SW_SPST, U1 TLV61070ADBV, U2 TSOP382xx, U3 TSOP382xx, U4 DRV8210DRLR, U5 BQ21040DBV, U6 ATtiny1604-SS, U7 Opamp_Dual, U8 DRV8210DRLR, X1 ASCO

Commit message: commit
Parts:
- added D8: D_Schottky, symbol Device:D_Schottky
Connections:
- net PA3: now also D8.1 (K); no longer X1.3 (OUT)
- new net: D8.2 (A), X1.3 (OUT)
Changed lines of the file:
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@@
 	(wire
 		(pts
-			(xy 48.26 91.44) (xy 53.34 91.44)
+			(xy 48.26 91.44) (xy 54.61 91.44)
 		)
 		(stroke
@@
 	(wire
 		(pts
+			(xy 62.23 91.44) (xy 66.04 91.44)
+		)
+		(stroke
+			(width 0)
+			(type default)
+		)
+	)
+	(wire
+		(pts
 			(xy 72.39 124.46) (xy 69.85 124.46)
 		)
@@
 	)
 	(label "PA3"
-		(at 53.34 91.44 180)
+		(at 66.04 91.44 180)
 		(effects
 			(font
@@
 	)
 	(symbol
+		(lib_id "Device:D_Schottky")
+		(at 58.42 91.44 180)
+		(unit 1)
+		(exclude_from_sim no)
+		(in_bom yes)
+		(on_board yes)
+		(dnp no)
+		(fields_autoplaced yes)
+		(property "Reference" "D8"
+			(at 58.7375 85.09 0)
+			(effects
+				(font
+					(size 1.27 1.27)
+				)
+			)
+		)
+		(property "Value" "D_Schottky"
+			(at 58.7375 87.63 0)
+			(effects
+				(font
+					(size 1.27 1.27)
+				)
+			)
+		)
+		(property "Footprint" ""
+			(at 58.42 91.44 0)
+			(effects
+				(font
+					(size 1.27 1.27)
+				)
+				(hide yes)
+			)
+		)
+		(property "Datasheet" "~"
+			(at 58.42 91.44 0)
+			(effects
+				(font
+					(size 1.27 1.27)
+				)
+				(hide yes)
+			)
+		)
+		(property "Description" "Schottky diode"
+			(at 58.42 91.44 0)
+			(effects
+				(font
+					(size 1.27 1.27)
+				)
+				(hide yes)
+			)
+		)
+		(pin "2"
+		)
+		(pin "1"
+		)
+		(instances
+			(project ""
+				(path "/bfbac227-b3e4-47e8-9776-0e31b83cca14"
+					(reference "D8")
+					(unit 1)
+				)
+			)
+		)
+	)
+	(symbol
 		(lib_id "power:GND")
 		(at 52.07 154.94 0)
@@
 	)
 	(symbol
-		(lib_name "Driver_Motor:DRV8210DRLR")
 		(lib_id "Driver_Motor:DRV8210DRLR")
 		(at 60.96 151.13 0)
@@
 	)
 	(symbol
-		(lib_name "Driver_Motor:DRV8210DRLR")
 		(lib_id "Driver_Motor:DRV8210DRLR")
 		(at 60.96 125.73 0)

Commit message: commit
Parts:
- U4, U8: footprint (none) -> Package_TO_SOT_SMD:SOT-563
Connections:
- net PA0: now also U8. (OUT2); no longer U4. (VM)
- net PA1: now also U8. (OUT2); no longer U4. (VM)
- net PB2: now also U4. (OUT2); no longer U8. (VM)
- net PB3: now also U4. (OUT2); no longer U8. (VM)
- net at M1.1 (+): now also U4. (OUT2); no longer U8. (VM)
- net at M1.2 (-): now also U4. (OUT2); no longer U8. (VM)
- net at M2.1 (+): now also U8. (OUT2); no longer U4. (VM)
- net at M2.2 (-): now also U8. (OUT2); no longer U4. (VM)
Other:
- moved on the sheet: C2, C3, D4, D5, R11, R12, U7A, U7B, U7C

Commit message: commit
Parts:
- removed D8: D_Schottky, symbol Device:D_Schottky
- removed U7: Opamp_Dual, symbol Device:Opamp_Dual
- removed X1: ASCO, Oscillator:Oscillator_SMD_Abracon_ASCO-4Pin_1.6x1.2mm, symbol Oscillator:ASCO
- added U7: LMV358, Package_SO:VSSOP-8_3x3mm_P0.65mm, symbol Amplifier_Operational:LMV358
- added XC4, XC5, XC6: 10u, symbol Device:C_Small
- C2, C3: value C -> 4.3p
- D1, D2: value LED -> IRLED
- D4, D5: value D_Photo -> VTP9812FH; footprint (none) -> Capacitor_THT:CP_Radial_D5.0mm_P2.50mm
- L1: value L -> 2.2u
- R1: value R -> 180k
- R11, R12: value R -> 1.24M
- R2: value R -> 20k
- R3, R8: value R -> 1.2k
- R4: value R -> 7.32k
- R6, R7: value R -> 200
- SW1: value SW_SPST -> SPST
- XC1: renamed from C1; value C -> 10u
- renumbered C4 to XC4, C5 to XC5
Connections:
- net +5V: now also U7.8 (V+), XC4.1
- net +BATT: now also XC6.1
- net GND: now also U7.2 (-), U7.4 (V-), U7.6 (-), XC4.2, XC5.2, XC6.2
- net PA4: now also U7.1
- net PA5: now also U7.7
- net VBUS: now also XC5.1
- net at C3.1, D4.1 (K), R11.1: now also U7.3 (+)
- net at C2.1, D5.1 (K), R12.1: now also U7.5 (+)
- no-connect marks 2 -> 1
Other:
- moved on the sheet: XC1

Commit message: commit
Parts:
- removed D2: IRLED, symbol Device:LED
- removed D4, D5: VTP9812FH, Capacitor_THT:CP_Radial_D5.0mm_P2.50mm, symbol Device:D_Photo
- removed M1: Motor_DC, symbol Motor:Motor_DC
- removed R7: 200, symbol Device:R_Small_US
- removed SW1: SPST, symbol Switch:SW_SPST
- removed U2, U3: TSOP382xx, OptoDevice:Vishay_MINICAST-3Pin, symbol Interface_Optical:TSOP382xx
- added C3: 47u, Capacitor_THT:CP_Radial_D5.0mm_P2.00mm, symbol Device:C_Polarized_Small_US
- added D11, D12: VTP9812FH, Capacitor_THT:CP_Radial_D5.0mm_P2.50mm, symbol Device:D_Photo
- added D3: IRLED, LED_THT:LED_D5.0mm, symbol Device:LED
- added D7, D8: LED, LED_SMD:LED_0805_2012Metric_Pad1.15x1.40mm_HandSolder, symbol Device:LED
- added J10: motor_right_m, symbol Connector_Generic:Conn_01x02
- added J11: rx_right_f, symbol Connector_Generic:Conn_01x04
- added J12: rx_left_f, symbol Connector_Generic:Conn_01x04
- added J13: tx_left_m, symbol Connector_Generic:Conn_01x02
- added J14: tx_right_m, symbol Connector_Generic:Conn_01x02
- added J3: tx_left_f, symbol Connector_Generic:Conn_01x02
- added J4: tx_right_f, symbol Connector_Generic:Conn_01x02
- added J5: rx_left_m, symbol Connector_Generic:Conn_01x04
- added J6: rx_right_m, symbol Connector_Generic:Conn_01x04
- added J7: motor_left_m, symbol Connector_Generic:Conn_01x02
- added J8: motor_left_f, symbol Connector_Generic:Conn_01x02
- added J9: motor_right_f, symbol Connector_Generic:Conn_01x02
- added M3: Motor_DC, symbol Motor:Motor_DC
- added Q2, Q3: T2N7002AK, Package_TO_SOT_SMD:SOT-23, symbol Transistor_FET:T2N7002AK
- added R15, R16: 1.2k, Resistor_SMD:R_0603_1608Metric_Pad0.98x0.95mm_HandSolder, symbol Device:R_Small_US
- added R5: 200, Resistor_SMD:R_0603_1608Metric_Pad0.98x0.95mm_HandSolder, symbol Device:R_Small_US
- added SW1: ANT11SF1CQE, symbol Switch:SW_SPDT
- added U10, U9: TSOP382xx, OptoDevice:Vishay_MINICAST-3Pin, symbol Interface_Optical:TSOP382xx
- added XC7, XC8, XC9: 0.1u, Capacitor_SMD:C_0603_1608Metric_Pad1.08x0.95mm_HandSolder, symbol Device:C_Small
- C1: renamed from C3; footprint (none) -> Capacitor_SMD:C_0603_1608Metric_Pad1.08x0.95mm_HandSolder
- C2, XC6: footprint (none) -> Capacitor_SMD:C_0603_1608Metric_Pad1.08x0.95mm_HandSolder
- D2: renamed from D1; footprint (none) -> LED_THT:LED_D5.0mm
- D5: renamed from D3; footprint (none) -> LED_SMD:LED_0805_2012Metric_Pad1.15x1.40mm_HandSolder
- D6: footprint (none) -> LED_SMD:LED_0805_2012Metric_Pad1.15x1.40mm_HandSolder
- J2: renamed from J1; footprint (none) -> Connector_USB:USB_C_Receptacle_HRO_TYPE-C-31-M-17
- L1: value 2.2u -> 2.2u, 2A; footprint (none) -> Inductor_SMD:L_1008_2520Metric_Pad1.43x2.20mm_HandSolder
- R1: renamed from R11; footprint (none) -> Resistor_SMD:R_0603_1608Metric_Pad0.98x0.95mm_HandSolder
- R10: renamed from R1; footprint (none) -> Resistor_SMD:R_0603_1608Metric_Pad0.98x0.95mm_HandSolder
- R11: renamed from R2; footprint (none) -> Resistor_SMD:R_0603_1608Metric_Pad0.98x0.95mm_HandSolder
- R12: renamed from R14; footprint (none) -> Resistor_SMD:R_0603_1608Metric_Pad0.98x0.95mm_HandSolder
- R13: footprint (none) -> Resistor_SMD:R_0603_1608Metric_Pad0.98x0.95mm_HandSolder
- R14: renamed from R3; footprint (none) -> Resistor_SMD:R_0603_1608Metric_Pad0.98x0.95mm_HandSolder
- R2: renamed from R6; footprint (none) -> Resistor_SMD:R_0603_1608Metric_Pad0.98x0.95mm_HandSolder
- R3: renamed from R9; footprint (none) -> Resistor_SMD:R_0603_1608Metric_Pad0.98x0.95mm_HandSolder
- R4: renamed from R10; footprint (none) -> Resistor_SMD:R_0603_1608Metric_Pad0.98x0.95mm_HandSolder
- R6: renamed from R12; footprint (none) -> Resistor_SMD:R_0603_1608Metric_Pad0.98x0.95mm_HandSolder
- R7: renamed from R8; footprint (none) -> Resistor_SMD:R_0603_1608Metric_Pad0.98x0.95mm_HandSolder
- R8: renamed from R4; footprint (none) -> Resistor_SMD:R_0603_1608Metric_Pad0.98x0.95mm_HandSolder
- R9: renamed from R5; footprint (none) -> Resistor_SMD:R_0603_1608Metric_Pad0.98x0.95mm_HandSolder
- XC1, XC5: renamed from XC4; footprint (none) -> Capacitor_SMD:C_0603_1608Metric_Pad1.08x0.95mm_HandSolder
- XC2, XC3: renamed from XC5; footprint (none) -> Capacitor_SMD:C_0603_1608Metric_Pad1.08x0.95mm_HandSolder
- XC4: renamed from XC1; footprint (none) -> Capacitor_SMD:C_0603_1608Metric_Pad1.08x0.95mm_HandSolder
- renumbered J2 to J1, U6 to U1, U8 to U2, U4 to U3, U7 to U4, U5 to U7, U1 to U8
Connections:
- net +5V: now also J13.2 (Pin_2), J14.2 (Pin_2), J5.1 (Pin_1), J6.1 (Pin_1), R15.1, R16.1, XC9.1; no longer R2.1
- net +BATT: now also C3.1, SW1.1 (A), XC7.1, XC8.1
- net GND: now also C3.2, J5.4 (Pin_4), J6.4 (Pin_4), Q2.2 (S), Q3.2 (S), XC7.2, XC8.2, XC9.2
- net PA6: now also J5.2 (Pin_2), Q2.1 (G)
- net PA7: now also J6.2 (Pin_2), Q3.1 (G)
- net tx_cathode: now reaches D5.1 (K), Q1.3 (D)
- net tx_cathode: now also J13.1 (Pin_1), J14.1 (Pin_1); no longer D2.1 (K)
- net IVL_left: now reaches C1.1, R1.1, U4.3 (+)
- net IVL_left: now also J5.3 (Pin_3)
- net IVL_right: now reaches C2.1, R6.1, U4.5 (+)
- net IVL_right: now also J6.3 (Pin_3)
- net at BT1.1 (+): now also SW1.2 (B)
- net at M2.1 (+): now also J8.1 (Pin_1); no longer U2. (OUT2)
- net at M2.2 (-): now also J8.2 (Pin_2); no longer U2. (OUT2)
- net PB1: no longer names the net of U1.8 (PB1)
- new net: D2.1 (K), J3.1 (Pin_1)
- new net: D12.1 (K), J12.3 (Pin_3)
- new net: D12.2 (A), J12.4 (Pin_4), U10.2 (GND)
- new net: D8.2 (A), R16.2
- new net: J12.1 (Pin_1), U10.3 (Vs)
- new net: J12.2 (Pin_2), U10.1 (OUT)
- new net: J3.2 (Pin_2), R2.1
- new net: D3.1 (K), J4.1 (Pin_1)
- new net: D3.2 (A), R5.2
- new net: J10.1 (Pin_1), U3. (OUT2)
- new net: J10.2 (Pin_2), U3. (OUT2)
- new net: J4.2 (Pin_2), R5.1
- new net: J11.2 (Pin_2), U9.1 (OUT)
- new net: D11.2 (A), J11.4 (Pin_4), U9.2 (GND)
- new net: J11.1 (Pin_1), U9.3 (Vs)
- new net: J7.1 (Pin_1), U2. (OUT2)
- new net: J7.2 (Pin_2), U2. (OUT2)
- new net: J9.1 (Pin_1), M3.1 (+)
- new net: J9.2 (Pin_2), M3.2 (-)
- new net: D11.1 (K), J11.3 (Pin_3)
- new net: D8.1 (K), Q3.3 (D)
- new net: D7.2 (A), R15.2
- new net: D7.1 (K), Q2.3 (D)
- no-connect marks 1 -> 3
Other:
- note added: "Battery Management"
- note added: "Controller"
- note added: "Infrared & Visible Light Receivers"
- note added: "Infrared Transmitters"
- note added: "Motor Drivers"
- note added: "Power"
- title: (none) -> Robo-Roach v1.0
- moved on the sheet: BT1, C1, C2, D2, D5, D6, J1, J2, L1, Q1, R1, R10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
