File: robo-roach-v1.0.kicad_sch (KiCad schematic)
At the start: 66 parts, among them J1 Prog, J10 motor_right_m, J11 rx_right_f, J12 rx_left_f, J13 tx_left_m, J14 tx_right_m, J2 USB_C_Receptacle_PowerOnly_6P, J3 tx_left_f, J4 tx_right_f, J5 rx_left_m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

Commit message: commit
Parts:
- J1: footprint (none) -> Connector_IDC:IDC-Header_2x03_P2.54mm_Vertical
Changed lines of the file:
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@@
 			)
 		)
-		(property "Footprint" ""
+		(property "Footprint" "Connector_IDC:IDC-Header_2x03_P2.54mm_Vertical"
 			(at 72.39 88.9 0)
 			(effects

Commit message: commit
Parts:
- added H1, H2, H3: M2, MountingHole:MountingHole_2.2mm_M2_DIN965_Pad, symbol Mechanical:MountingHole_Pad
- added TP1: +5V, TestPoint:TestPoint_THTPad_D1.0mm_Drill0.5mm, symbol Connector:TestPoint
- added TP2: +BATT, TestPoint:TestPoint_THTPad_D1.0mm_Drill0.5mm, symbol Connector:TestPoint
- added TP3: VBUS, TestPoint:TestPoint_THTPad_D1.0mm_Drill0.5mm, symbol Connector:TestPoint
- added TP4: VL_R, TestPoint:TestPoint_THTPad_D1.0mm_Drill0.5mm, symbol Connector:TestPoint
- added TP5: VL_L, TestPoint:TestPoint_THTPad_D1.0mm_Drill0.5mm, symbol Connector:TestPoint
- added TP6: IR_L, TestPoint:TestPoint_THTPad_D1.0mm_Drill0.5mm, symbol Connector:TestPoint
- added TP7: IR_R, TestPoint:TestPoint_THTPad_D1.0mm_Drill0.5mm, symbol Connector:TestPoint
- added TP8: GND, TestPoint:TestPoint_THTPad_D1.0mm_Drill0.5mm, symbol Connector:TestPoint
- BT1, J10, J13, J14, J3, J4, J7, J8, J9: footprint (none) -> robo-roach:LHA-02-TS
- J1: footprint Connector_IDC:IDC-Header_2x03_P2.54mm_Vertical -> robo-roach:SWR204-NRTN-D03-ST-GA
- J11, J12, J5, J6: footprint (none) -> robo-roach:LHA-04-TS
- SW1: footprint (none) -> robo-roach:ANT11SECQE
Connections:
- net +5V: now also TP1.1
- net +BATT: now also U2.6 (VM), U3.6 (VM), TP2.1; no longer U2. (OUT2), U3. (OUT2)
- net GND: now also U2.3 (GND), U3.3 (GND), H1.1, H2.1, H3.1, TP8.1; no longer U2. (OUT2), U3. (OUT2)
- net PA0: no longer U2. (OUT2)
- net PA1: no longer U2. (OUT2)
- net PA3: now also R3.1
- net PA4: now also TP5.1
- net PA5: now also TP4.1
- net PA6: now also TP6.1
- net PA7: now also TP7.1
- net PB0: now also U2.1 (IN1); no longer R3.1
- net PB2: now also U3.1 (IN1); no longer U3. (OUT2)
- net PB3: now also U3.2 (IN2); no longer U3. (OUT2)
- net VBUS: now also TP3.1
- net PB1: now reaches U1.8 (PB1)
- net PB1: now also U2.2 (IN2)
- net at J10.1 (Pin_1): now also U3.5 (OUT1); no longer U3. (OUT2)
- net at J10.2 (Pin_2): now also U3.4 (OUT2); no longer U3. (OUT2)
- net at J7.1 (Pin_1): now also U2.5 (OUT1); no longer U2. (OUT2)
- net at J7.2 (Pin_2): now also U2.4 (OUT2); no longer U2. (OUT2)
- no-connect marks 3 -> 2

Commit message: commit
Parts:
- D11, D12: footprint Capacitor_THT:CP_Radial_D5.0mm_P2.50mm -> LED_THT:LED_D5.0mm
- J8, J9: footprint robo-roach:LHA-02-TS -> (none)
- U10, U9: footprint OptoDevice:Vishay_MINICAST-3Pin -> robo-roach:TSOP38336_Right_Angled
Changed lines of the file:
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@@
 			)
 		)
-		(property "Footprint" "robo-roach:LHA-02-TS"
+		(property "Footprint" ""
 			(at 260.35 208.28 0)
 			(effects
@@
 			)
 		)
-		(property "Footprint" "Capacitor_THT:CP_Radial_D5.0mm_P2.50mm"
+		(property "Footprint" "LED_THT:LED_D5.0mm"
 			(at 87.63 129.54 0)
 			(effects
@@
 			)
 		)
-		(property "Footprint" "OptoDevice:Vishay_MINICAST-3Pin"
+		(property "Footprint" "robo-roach:TSOP38336_Right_Angled"
 			(at 115.57 213.995 0)
 			(effects
@@
 			)
 		)
-		(property "Footprint" "Capacitor_THT:CP_Radial_D5.0mm_P2.50mm"
+		(property "Footprint" "LED_THT:LED_D5.0mm"
 			(at 87.63 205.74 0)
 			(effects
@@
 			)
 		)
-		(property "Footprint" "robo-roach:LHA-02-TS"
+		(property "Footprint" ""
 			(at 260.35 246.38 0)
 			(effects
@@
 			)
 		)
-		(property "Footprint" "OptoDevice:Vishay_MINICAST-3Pin"
+		(property "Footprint" "robo-roach:TSOP38336_Right_Angled"
 			(at 115.57 137.795 0)
 			(effects

Commit message: commit
Connections:
- net PA1 is gone; now on net +BATT: J1.5 (Pin_5), U1.11 (PA1)
Changed lines of the file:
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@@
 	(wire
 		(pts
-			(xy 88.9 40.64) (xy 93.98 40.64)
+			(xy 88.9 40.64) (xy 96.52 40.64)
 		)
 		(stroke
@@
 					(unit 1)
 				)
+			)
+		)
+	)
+	(symbol
+		(lib_id "power:+BATT")
+		(at 96.52 40.64 0)
+		(unit 1)
+		(exclude_from_sim no)
+		(in_bom yes)
+		(on_board yes)
+		(dnp no)
+		(fields_autoplaced yes)
+		(property "Reference" "#PWR064"
+			(at 96.52 44.45 0)
+			(effects
+				(font
+					(size 1.27 1.27)
+				)
+				(hide yes)
+			)
+		)
+		(property "Value" "+BATT"
+			(at 96.52 35.56 0)
+			(effects
+				(font
+					(size 1.27 1.27)
+				)
+			)
+		)
+		(property "Footprint" ""
+			(at 96.52 40.64 0)
+			(effects
+				(font
+					(size 1.27 1.27)
+				)
+				(hide yes)
+			)
+		)
+		(property "Datasheet" ""
+			(at 96.52 40.64 0)
+			(effects
+				(font
+					(size 1.27 1.27)
+				)
+				(hide yes)
+			)
+		)
+		(property "Description" "Power symbol creates a global label with name \"+BATT\""
+			(at 96.52 40.64 0)
+			(effects
+				(font
+					(size 1.27 1.27)
+				)
+				(hide yes)
+			)
+		)
+		(pin "1"
+		)
+		(instances
+			(project "robo-roach-v1.0"
+				(path "/bfbac227-b3e4-47e8-9776-0e31b83cca14"
+					(reference "#PWR064")
+					(unit 1)
+				)
