File: robo-roach-v1.0.kicad_pcb (KiCad board)
At the start: 4 copper layers, 38.1 x 61 mm, 61 parts, among them J1 Prog, J10 motor_right_m, J13 tx_left_m, J14 tx_right_m, J2 USB_C_Receptacle_PowerOnly_6P, J5 rx_left_m, J6 rx_right_m, J7 motor_left_m, Q1 T2N7002AK, Q2 T2N7002AK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

Commit message: commit
Routing:
- net +BATT: track 0.76 -> 4.54 mm, vias 11 -> 10
Other:
- board text added: "CHG"
- board text added: "RX_L"
- board text added: "RX_R"
- board text added: "TX"
Changed lines of the file:
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@@
 		(at 161.29 106.68 -90)
 		(property "Reference" "J7"
-			(at -3.81 0 0)
+			(at 3.556 0 0)
 			(unlocked yes)
 			(layer "F.SilkS")
@@
 		(at 161.29 114.3 -90)
 		(property "Reference" "J13"
-			(at -3.81 0 0)
+			(at 3.556 0 0)
 			(unlocked yes)
 			(layer "F.SilkS")
@@
 		(at 130.81 114.3 -90)
 		(property "Reference" "J14"
-			(at -3.81 0 0)
+			(at 3.556 0 0)
 			(unlocked yes)
 			(layer "F.SilkS")
@@
 		(at 130.81 106.68 90)
 		(property "Reference" "J10"
-			(at 3.81 0.0775 0)
+			(at -3.556 0 0)
 			(unlocked yes)
 			(layer "F.SilkS")
@@
 		)
 	)
+	(gr_text "CHG"
+		(at 127.254 126.492 0)
+		(layer "F.SilkS")
+		(effects
+			(font
+				(size 1 1)
+				(thickness 0.15)
+			)
+			(justify left bottom)
+		)
+	)
+	(gr_text "RX_R"
+		(at 127.127 102.362 0)
+		(layer "F.SilkS")
+		(effects
+			(font
+				(size 1 1)
+				(thickness 0.15)
+			)
+			(justify left bottom)
+		)
+	)
+	(gr_text "RX_L"
+		(at 161.163 102.362 0)
+		(layer "F.SilkS")
+		(effects
+			(font
+				(size 1 1)
+				(thickness 0.15)
+			)
+			(justify left bottom)
+		)
+	)
+	(gr_text "TX"
+		(at 145.034 117.983 0)
+		(layer "F.SilkS")
+		(effects
+			(font
+				(size 1 1)
+				(thickness 0.15)
+			)
+			(justify left bottom)
+		)
+	)
 	(segment
 		(start 138.725 134.96)
@@
 		(net 7)
 	)
-	(via
-		(at 128.905 122.165)
-		(size 0.4)
-		(drill 0.3)
-		(layers "F.Cu" "B.Cu")
+	(segment
+		(start 154.8325 115.57)
+		(end 154.8325 119.3525)
+		(width 1.016)
+		(layer "F.Cu")
 		(net 7)
 	)
 	(via
-		(at 154.8325 115.57)
+		(at 128.905 122.165)
 		(size 0.4)
 		(drill 0.3)

Commit message: commit
Routing:
- net /PB3: track 8.74 -> 10.1 mm
- net /PB2: track 7.09 -> 8.13 mm
- net GND: vias 28 -> 49
- net +BATT: vias 10 -> 22
- added copper zone on F.Cu, net +BATT

Commit message: commit
Parts:
- added D11: VTP9812FH, LED_THT:LED_D5.0mm, F.Cu at (173.4, 90.8)
- added D12: VTP9812FH, LED_THT:LED_D5.0mm, F.Cu at (189.9, 90.8)
- added D2: IRLED, LED_THT:LED_D5.0mm, F.Cu at (135.2, 67.3)
- added D3: IRLED, LED_THT:LED_D5.0mm, F.Cu at (155.6, 67.3)
- added J11: rx_right_f, robo-roach:LHA-04-TS, B.Cu at (177.2, 94.6)
- added J12: rx_right_f, robo-roach:LHA-04-TS, B.Cu at (193.7, 94.6)
- added J3: tx_left_f, robo-roach:LHA-02-TS, B.Cu at (136.5, 71.1)
- added J4: tx_right_f, robo-roach:LHA-02-TS, B.Cu at (156.8, 71.1)
- added R2: 200, Resistor_SMD:R_0603_1608Metric_Pad0.98x0.95mm_HandSolder, F.Cu at (141.0, 68.6)
- added R5: 200, Resistor_SMD:R_0603_1608Metric_Pad0.98x0.95mm_HandSolder, F.Cu at (161.3, 68.6)
- added U10: TSOP382xx, robo-roach:TSOP38336_Right_Angled, F.Cu at (189.9, 102.4)
- added U9: TSOP382xx, robo-roach:TSOP38336_Right_Angled, F.Cu at (173.4, 102.4)
Routing:
- net Net-(D11-A): track 0.00 -> 22.1 mm
- net Net-(D12-A): track 0.00 -> 22.1 mm
- net Net-(J12-Pin_2): track 0.00 -> 9.17 mm
- net Net-(J11-Pin_2): track 0.00 -> 9.17 mm
- net Net-(D11-K): track 0.00 -> 4.86 mm
- net Net-(D12-K): track 0.00 -> 4.86 mm
- net Net-(J12-Pin_1): track 0.00 -> 4.53 mm
- net Net-(J11-Pin_1): track 0.00 -> 4.53 mm
- net Net-(J3-Pin_2): track 0.00 -> 3.85 mm
- net Net-(J4-Pin_2): track 0.00 -> 3.85 mm
- net Net-(D3-K): track 0.00 -> 3.81 mm
- net Net-(D2-K): track 0.00 -> 3.81 mm
- net Net-(D3-A): track 0.00 -> 3.33 mm
- net Net-(D2-A): track 0.00 -> 3.32 mm
- net +BATT: vias 22 -> 20
Other:
- board size 38.1 x 61 mm -> 70.5 x 74.9 mm

Commit message: commit
Connections:
- J1 pad 5: /PA1 -> +BATT
- U1 pad 11: /PA1 -> +BATT
Routing:
- net /PA1: track 3.78 -> 0.00 mm
- net +BATT: track 4.54 -> 8.32 mm, vias 20 -> 21
